Commit message: Adiciona sensor UWB simulado (ativação apenas, fora da localização)
Adiciona uma tag UWB no robô e uma âncora por planta (10 no total, a 1.0 m
de altura) usando o plugin externo uwb_gazebosensorplugins (AUVSL). O
sensor publica ranging real (/gtec/toa/ranging) com modelo de LOS/NLOS,
mas não participa do EKF nem de nenhuma outra parte da localização.

Corrige também um bug de fusão (lumping) do link da tag na conversão
URDF->SDF, que fazia a origem do raio de UWB ficar dentro da própria
colisão do robô e bloquear todo o ranging — resolvido com tag_z_offset.

File: urdf/agrobot.gazebo.xacro (robot description, xacro)
@@ -122,3 +122,32 @@
        adicionado de propósito — ver seção 4.2(g) do prompt. Pose real,
        quando precisar, vem de /gazebo/model_states. -->
+  <!-- Tag UWB — plugin externo (uwb_gazebosensorplugins, clonado à parte
+       em ~/catkin_ws/src/, não faz parte deste pacote). Só ativa o sensor
+       simulado (publica ranging em /gtec/toa/ranging e /gtec/toa/anchors);
+       NÃO entra no EKF nem em nenhuma outra parte da localização — por
+       pedido explícito, isso fica de fora por enquanto.
+       tag_z_offset=0.3: o Gazebo funde (lump) o uwb_tag_link — vazio, sem
+       geometria — dentro do base_link ao converter URDF->SDF (confirmado
+       no log ~/.gazebo/server-*/default.log: "Tag link Is NULL"); as tags
+       <preserveFixedJoint>/<disableFixedJointLumping> no
+       agrobot.urdf.xacro não evitaram isso nesta versão do Gazebo/ROS. Com
+       o link fundido, o plugin usa a pose do MODELO inteiro como origem do
+       raio de LOS — bem próxima da própria caixa de colisão do chassi, o
+       que fazia todo raio bater no próprio robô e nenhum ranging nunca era
+       publicado (testado e confirmado com all_los=1: só aí o ranging
+       aparecia). O tag_z_offset levanta essa origem 0.3 m, para fora do
+       chassi, e resolve isso sem precisar consertar o lumping —
+       comportamento de LOS/NLOS real (raycasting) volta a funcionar. -->
+  <gazebo>
+    <plugin name="libgtec_uwb_plugin" filename="libgtec_uwb_plugin.so">
+      <update_rate>10</update_rate>
+      <nlosSoftWallWidth>0.1</nlosSoftWallWidth>
+      <tag_z_offset>0.3</tag_z_offset>
+      <tag_link>uwb_tag_link</tag_link>
+      <anchor_prefix>uwb_anchor</anchor_prefix>
+      <all_los>false</all_los>
+      <tag_id>0</tag_id>
+      <return_angle>true</return_angle>
+    </plugin>
+  </gazebo>
 </robot>

File: urdf/agrobot.urdf.xacro (robot description, xacro)
@@ -120,4 +120,24 @@
   <link name="imu_link"/>
   <!--
+    Tag UWB (plugin externo uwb_gazebosensorplugins/gtec_uwb_plugin, ver
+    agrobot.gazebo.xacro). Fixa no topo do chassi, só para ter uma origem
+    de medição de distância às âncoras do mundo — não participa do EKF.
+  -->
+  <joint name="uwb_tag_joint" type="fixed">
+    <parent link="base_link"/>
+    <child link="uwb_tag_link"/>
+    <origin xyz="-0.032 0 0.15" rpy="0 0 0"/>
+  </joint>
+  <link name="uwb_tag_link"/>
+  <!-- Sem isso, o Gazebo funde (lump) o uwb_tag_link — vazio, sem
+       geometria — dentro do base_link na conversão URDF->SDF, e
+       _parent->GetLink("uwb_tag_link") no plugin retorna NULL (confirmado
+       no log ~/.gazebo/server-*/default.log: "Tag link Is NULL"). O mesmo
+       aviso está no README do plugin para as âncoras. -->
+  <gazebo reference="uwb_tag_joint">
+    <preserveFixedJoint>true</preserveFixedJoint>
+    <disableFixedJointLumping>true</disableFixedJointLumping>
+  </gazebo>
+  <!--
     base_scan: link, joint e malha do LDS-01 mantidos de propósito (ver seção 4.1).
     Isso preserva massa e inércia idênticas ao burger real. O que desaparece é
